Commit message: new update yaml param

File: tifa_bot/description/robot_core.xacro (robot description, xacro)
@@ -19,4 +19,12 @@
     <!-- BASE LINK -->
     <link name="base_link">
+    </link>
+    <!-- BASE FOOTPRINT     -->
+    <joint name="base_footprint_joint" type="fixed">
+        <parent link="base_link"/>
+        <child link="base_footprint"/>
+        <origin xyz="0 0 0" rpy="0 0 0"/>
+    </joint>
+    <link name="base_footprint">
     </link>
     <!-- CHASSIS LINK  -->
@@ -53,5 +61,5 @@
         <parent link="base_link"/>
         <child link="left_wheel"/>
-        <origin xyz="0.0 0.275 0.0" rpy="-${pi/2} 0 0"/>
+        <origin xyz="0.0 0.2125 0.0" rpy="-${pi/2} 0 0"/>
         <axis xyz="0.0 0.0 1.0"/>
     </joint>
@@ -81,5 +89,5 @@
         <parent link="base_link"/>
         <child link="right_wheel"/>
-        <origin xyz="0.0 -0.275 0.0" rpy="${pi/2} 0 0"/>
+        <origin xyz="0.0 -0.2125 0.0" rpy="${pi/2} 0 0"/>
         <axis xyz="0.0 0.0 -1.0"/>
     </joint>
